File: hardware/two_comparator_effect.kicad_pcb (KiCad board)
At the start: 2 copper layers, 100 x 35 mm, 34 parts, among them J1 rca, J2 rca, J3 Barrel_Jack, Q1 2N3904, SW1 SW_DPDT_x2, U1 LM339, U2 LM317

Commit message: refactor files
Parts:
- J3: footprint Connector_BarrelJack:BarrelJack_Horizontal -> lib:BarrelJack_Horizontal
