File: hardware/two_comparator_effect.kicad_pcb (KiCad board)
At the start: 2 copper layers, 100 x 35 mm, 34 parts, among them J1 rca, J2 rca, J3 Barrel_Jack, Q1 2N3904, SW1 SW_DPDT_x2, U1 LM339, U2 LM317

Commit message: update bom
Other:
- board text added: "JLCJLCJLCJLC"

Commit message: update booklet
Parts:
- R1, R5: value 4.7k -> 3k
- R4, R7: value 1.2k -> 910
Connections:
- U1 pad 14: Net-(U1-Pad14) -> unconnected-(U1-Pad14)
- U1 pad 8: Net-(U1-Pad8) -> unconnected-(U1-Pad8)
- U1 pad 9: Net-(U1-Pad9) -> unconnected-(U1-Pad9)
Other:
- net class Default removed
